File: hw/rascsi_2p4/USB_Conn.sch (KiCad schematic (older format))
At the start: 4 parts, among them J8 USB_B_Micro

Commit message: made 25pin and USB conn placeable by JLCPCB
Parts:
- J8: footprint SamacSys_Parts:U254051N4BH806 -> SamacSys_Parts:U254051N4BH806_JLCPCB_hand_mount
Changed lines of the file:
@@
 F 0 "J8" H 3350 2300 50  0000 C CNN
 F 1 "USB_B_Micro" H 3350 2200 50  0000 C CNN
-F 2 "SamacSys_Parts:U254051N4BH806" H 3050 2000 50  0001 C CNN
+F 2 "SamacSys_Parts:U254051N4BH806_JLCPCB_hand_mount" H 3050 2000 50  0001 C CNN
 F 3 "https://datasheet.lcsc.com/szlcsc/2002271812_XKB-Connectivity-U254-051N-4BH806_C319170.pdf" H 3050 2000 50  0001 C CNN
 F 4 "C319170" H 2900 2050 50  0001 C CNN "LCSC"
