File: hw/rascsi_2p4/Connectors.sch (KiCad schematic (older format))
At the start: 5 parts, among them J10 Conn_01x04_Male, J20 171826-4, J3 Conn_02x25_Odd_Even, J9 Conn_02x25_Odd_Even

Commit message: made 25pin and USB conn placeable by JLCPCB
Parts:
- J3: footprint Connector_PinHeader_2.54mm:PinHeader_2x25_P2.54mm_Vertical -> amiga:PinHeader_2x25_P2.54mm_Vertical_JLCPCB_hand_mount
Changed lines of the file:
@@
 F 0 "J3" H 3000 275 50  0000 C CNN
 F 1 "Conn_02x25_Odd_Even" H 3000 366 50  0000 C CNN
-F 2 "Connector_PinHeader_2.54mm:PinHeader_2x25_P2.54mm_Vertical" H 2950 1700 50  0001 C CNN
+F 2 "amiga:PinHeader_2x25_P2.54mm_Vertical_JLCPCB_hand_mount" H 2950 1700 50  0001 C CNN
 F 3 "https://datasheet.lcsc.com/szlcsc/1810221914_BOOMELE-Boom-Precision-Elec-C30006_C30006.pdf" H 2950 1700 50  0001 C CNN
 F 4 "C30006" H 2950 1700 50  0001 C CNN "LCSC"

Commit message: fixed part positioning at JLCPCB by removing 2x25 Pin Header from Handmount
Parts:
- J3: footprint amiga:PinHeader_2x25_P2.54mm_Vertical_JLCPCB_hand_mount -> Connector_PinHeader_2.54mm:PinHeader_2x25_P2.54mm_Vertical
Changed lines of the file:
@@
 F 0 "J3" H 3000 275 50  0000 C CNN
 F 1 "Conn_02x25_Odd_Even" H 3000 366 50  0000 C CNN
-F 2 "amiga:PinHeader_2x25_P2.54mm_Vertical_JLCPCB_hand_mount" H 2950 1700 50  0001 C CNN
+F 2 "Connector_PinHeader_2.54mm:PinHeader_2x25_P2.54mm_Vertical" H 2950 1700 50  0001 C CNN
 F 3 "https://datasheet.lcsc.com/szlcsc/1810221914_BOOMELE-Boom-Precision-Elec-C30006_C30006.pdf" H 2950 1700 50  0001 C CNN
 F 4 "C30006" H 2950 1700 50  0001 C CNN "LCSC"
